File: pcb/40keyboardpico/40keyboardpico.kicad_pcb (KiCad board)
At the start: 2 copper layers, 76.2 x 76.2 mm, 48 parts, among them J1 Conn_01x04, J10 Conn_01x04, J11 AudioJack4, J2 Conn_01x04, J3 Conn_01x04, J4 Conn_01x04, J5 Conn_01x04, J6 Conn_01x04, J7 Conn_01x04, J8 Conn_01x04, J9 Conn_01x04, SW1 SW_Push, SW10 SW_Push, SW11 SW_Push, SW12 SW_Push, SW13 SW_Push, SW14 SW_Push, SW15 SW_Push, SW16 SW_Push, SW2 SW_Push, SW3 SW_Push, SW4 SW_Push, SW5 SW_Push, SW6 SW_Push, SW7 SW_Push, SW8 SW_Push, SW9 SW_Push, U1 Pico

Commit message: Add area ground.
Routing:
- net GND: vias 1 -> 2
- added copper zone on B.Cu, net GND
- added copper zone on F.Cu, net GND
Changed lines of the file:
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@@
     (thickness 1.6)
     (drawings 7)
-    (tracks 459)
+    (tracks 460)
     (zones 0)
     (modules 48)
@@
   (segment (start 160.885 94.845) (end 167.585 94.845) (width 0.25) (layer F.Cu) (net 41))
   (segment (start 158.115 92.075) (end 160.885 94.845) (width 0.25) (layer F.Cu) (net 41))
+  (via (at 147.955 153.035) (size 0.8) (drill 0.4) (layers F.Cu B.Cu) (net 41))
   (via (at 165.735 92.744999) (size 0.8) (drill 0.4) (layers F.Cu B.Cu) (net 42))
   (segment (start 170.534999 92.744999) (end 165.735 92.744999) (width 0.25) (layer B.Cu) (net 42))
@@
   (segment (start 156.845 111.125) (end 153.764999 114.205001) (width 0.25) (layer F.Cu) (net 44))
   (segment (start 148.59 115.57) (end 132.715 115.57) (width 0.25) (layer B.Cu) (net 44))
+  (zone (net 41) (net_name GND) (layer F.Cu) (hatch edge 0.508)
+    (connect_pads (clearance 0.508))
+    (min_thickness 0.254)
+    (fill yes (arc_segments 32) (thermal_gap 0.508) (thermal_bridge_width 0.508))
+    (polygon
+      (pts
+        (xy 189.23 157.48) (xy 113.03 157.48) (xy 113.03 81.28) (xy 189.23 81.28)
+      )
+    )
+  )
+  (zone (net 41) (net_name GND) (layer B.Cu) (hatch edge 0.508)
+    (connect_pads (clearance 0.508))
+    (min_thickness 0.254)
+    (fill yes (arc_segments 32) (thermal_gap 0.508) (thermal_bridge_width 0.508))
+    (polygon
+      (pts
+        (xy 189.23 157.48) (xy 113.03 157.48) (xy 113.03 81.28) (xy 189.23 81.28)
+      )
+    )
+  )
 )

Commit message: Send it to all pcb.
Parts:
- removed REF** (x4): PinHeader_1x01_P2.54mm_Vertical, Connector_PinHeader_2.54mm:PinHeader_1x01_P2.54mm_Vertical
Connections:
- U1 pad 13: Net-(U1-Pad13) -> GND
- U1 pad 18: Net-(U1-Pad18) -> GND
- U1 pad 23: Net-(U1-Pad23) -> GND
- U1 pad 28: Net-(U1-Pad28) -> GND
- U1 pad 3: Net-(U1-Pad3) -> GND
- U1 pad 33: Net-(U1-Pad33) -> GND
- U1 pad 8: Net-(U1-Pad8) -> GND
